File: design/AMS1117DC3V3/AMS1117DC3V3.kicad_pcb (KiCad board)
At the start: 2 copper layers, 25.8 x 11.1 mm, 1 part, among them U1 AMS1117-3.3

Commit message: final version
Parts:
- added C1: C, Capacitor_SMD:C_0603_1608Metric, F.Cu at (25.3, 25.3)
- added C2: C, Capacitor_SMD:C_0603_1608Metric, F.Cu at (27.7, 25.3)
- added C3: C, Capacitor_SMD:C_0603_1608Metric, F.Cu at (38.5, 25.3)
- added C4: C, Capacitor_SMD:C_0603_1608Metric, F.Cu at (40.9, 25.3)
- added D1: LED, LED_SMD:LED_1206_3216Metric, F.Cu at (25.6, 29.5)
- added J1: Conn_01x02, Connector_PinHeader_2.54mm:PinHeader_1x02_P2.54mm_Vertical, F.Cu at (21.7, 24.0)
- added J2: Conn_01x02, Connector_PinHeader_2.54mm:PinHeader_1x02_P2.54mm_Vertical, F.Cu at (44.0, 24.0)
- added R1: 1k, Resistor_SMD:R_1206_3216Metric, F.Cu at (39.0, 29.2)
Connections:
- U1 pad 1: unconnected-(U1-GND/ADJ-Pad1) -> GND
- U1 pad 2: unconnected-(U1-VOUT-Pad2) -> Vout
- U1 pad 3: unconnected-(U1-VIN-Pad3) -> Vin
Routing:
- net Vout: track 0.00 -> 23.5 mm
- net Net-(D1-A): track 0.00 -> 11.3 mm
- net GND: track 0.00 -> 1.08 mm, vias 0 -> 6
- net Vin: track 0.00 -> 0.74 mm
- added copper zone on B.Cu, net GND
- added copper zone on F.Cu, net GND
- added copper zone on F.Cu, net Vin
