File: design/AMS1117DC3V3/AMS1117DC3V3.kicad_sch (KiCad schematic)
At the start: 9 parts, among them J1 Conn_01x02_MountingPin, J2 Conn_01x02_MountingPin, U1 AMS1117-3.3

Commit message: final version
Parts:
- removed J1, J2: Conn_01x02_MountingPin, symbol Connector_Generic_MountingPin:Conn_01x02_MountingPin
- added J1, J2: Conn_01x02, Connector_PinHeader_2.54mm:PinHeader_1x02_P2.54mm_Vertical, symbol Connector_Generic:Conn_01x02
- C1, C2, C3, C4: footprint (none) -> Capacitor_SMD:C_0603_1608Metric
- D1: footprint (none) -> LED_SMD:LED_1206_3216Metric
- R1: value R -> 1k; footprint (none) -> Resistor_SMD:R_1206_3216Metric
Connections:
- net Vout: now reaches C3.1
- net Vout: now also C4.1, R1.1, U1.2 (VOUT), J2.1 (Pin_1)
- net GND: now reaches C3.2
- net GND: now also C1.2, C2.2, C4.2, D1.1 (K), U1.1 (GND/ADJ), J1.2 (Pin_2), J2.2 (Pin_2)
- net Vin: now reaches C1.1
- net Vin: now also C2.1, U1.3 (VIN), J1.1 (Pin_1)
- net at D1.2 (A): now also R1.2
Other:
- note added: "3.3V LDO Regulation"
- note added: "3.3V Output OK LED"
- note added: "Input connector"
- note added: "Output connector"
- company: (none) -> AvelTek
- title: (none) -> AMS117DC3V3
- moved on the sheet: C1, C2, C3, C4, D1, R1, U1
